File: pcb/simplekeyboard.kicad_pcb (KiCad board)
At the start: 2 copper layers, 145 parts, among them J1 USB_C_Receptacle_USB2.0_16P, SW1 SW_Push, SW10 SW_Push, SW11 SW_Push, SW12 SW_Push, SW13 SW_Push, SW14 SW_Push, SW15 SW_Push, SW16 SW_Push, SW17 SW_Push, SW18 SW_Push, SW19 SW_Push, SW2 SW_Push, SW20 SW_Push, SW21 SW_Push, SW22 SW_Push, SW23 SW_Push, SW24 SW_Push, SW25 SW_Push, SW26 SW_Push, SW27 SW_Push, SW28 SW_Push, SW29 SW_Push, SW3 SW_Push, SW30 SW_Push, SW31 SW_Push, SW32 SW_Push, SW33 SW_Push, SW34 SW_Push, SW35 SW_Push, SW36 SW_Push, SW37 SW_Push, SW38 SW_Push, SW39 SW_Push, SW4 SW_Push, SW40 SW_Push, SW41 SW_Push, SW42 SW_Push, SW43 SW_Push, SW44 SW_Push, SW45 SW_Push, SW46 SW_Push, SW47 SW_Push, SW48 SW_Push, SW49 SW_Push, SW5 SW_Push, SW50 SW_Push, SW51 SW_Push, SW52 SW_Push, SW53 SW_Push, SW54 SW_Push, SW55 SW_Push, SW56 SW_Push, SW57 SW_Push, SW58 SW_Push, SW59 SW_Push, SW6 SW_Push, SW60 SW_Push, SW61 SW_Push, SW62 SW_SPDT, SW63 SW_Push, SW7 SW_Push, SW8 SW_Push, SW9 SW_Push, U1 STM32F072CBT6, U2 USBLC6-2SC6, U3 LD39050PU33R

Commit message: Almost done PCB
Parts:
- C1, C2: footprint Capacitor_SMD:C_0805_2012Metric_Pad1.18x1.45mm_HandSolder -> Capacitor_SMD:C_0603_1608Metric
- C10, C11, C3, C4, C5, C6, C7, C8, C9: footprint Capacitor_SMD:C_0805_2012Metric_Pad1.18x1.45mm_HandSolder -> Capacitor_SMD:C_0603_1608Metric; moved to B.Cu
- D10, D11, D12, D13, D14, D15, D16, D17, D18, D19, D2, D20, D21, D22, D23, D24, D25, D26, D27, D28, D29, D3, D30, D31, D32, D33, D34, D35, D36, D37, D38, D39, D4, D40, D41, D42, D43, D44, D45, D46, D47, D48, D49, D5, D50, D51, D52, D53, D54, D55, D56, D57, D58, D59, D6, D60, D61, D7, D8, D9, SW62, SW63, TP1, TP2: moved to B.Cu
- R1, R2: footprint Resistor_SMD:R_0805_2012Metric_Pad1.20x1.40mm_HandSolder -> Resistor_SMD:R_0805_2012Metric
- R3: footprint Resistor_SMD:R_0805_2012Metric_Pad1.20x1.40mm_HandSolder -> Resistor_SMD:R_0805_2012Metric; moved to B.Cu
- moved D54 353.9 mm to (39.3, 108.3), turned to -90 degrees
- moved D42 339.6 mm to (48.8, 89.3), turned to -90 degrees
- moved D29 339.3 mm to (44.1, 70.2), turned to -90 degrees
- moved D15 336.3 mm to (41.7, 51.2), turned to -90 degrees
- moved D55 334.5 mm to (63.1, 108.3), turned to -90 degrees
- moved D2 318.2 mm to (56.0, 32.1), turned to -90 degrees
- moved D16 314.0 mm to (65.5, 51.2), turned to -90 degrees
- moved D30 313.9 mm to (70.2, 70.2), turned to -90 degrees
- moved D56 310.7 mm to (86.9, 108.3), turned to -90 degrees
- moved D43 309.3 mm to (79.8, 89.3), turned to -90 degrees
- moved D3 300.9 mm to (75.0, 32.1), turned to -90 degrees
- moved D17 296.6 mm to (84.5, 51.2), turned to -90 degrees
- moved D31 295.7 mm to (89.3, 70.2), turned to -90 degrees
- moved D44 291.0 mm to (98.8, 89.3), turned to -90 degrees
- moved TP1 284.2 mm to (57.2, 43.0), turned to 180 degrees
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Connections:
- net Net-(J1-D+-PadA6) renamed /REC_USB_D+
- net Net-(J1-D--PadA7) renamed /REC_USB_D-
Routing:
- net /Matrix/COL3: track 0.00 -> 115.4 mm
- net /Matrix/COL10: track 0.00 -> 96.3 mm
- net /Matrix/COL1: track 0.00 -> 93.2 mm
- net /Matrix/COL2: track 0.00 -> 91.0 mm
- net /Matrix/COL13: track 0.00 -> 89.0 mm
- net /Matrix/COL11: track 0.00 -> 85.5 mm
- net /Matrix/COL0: track 0.00 -> 85.1 mm
- net /Matrix/COL12: track 0.00 -> 81.1 mm
- net /Matrix/COL7: track 0.00 -> 67.0 mm
- net /Matrix/COL4: track 0.00 -> 67.0 mm
- net /Matrix/COL9: track 0.00 -> 67.0 mm
- net /Matrix/COL8: track 0.00 -> 67.0 mm
- net /Matrix/COL6: track 0.00 -> 67.0 mm
- net /Matrix/COL5: track 0.00 -> 67.0 mm
- net +3.3V: track 2.06 -> 58.2 mm
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
Commit message: Route diodes
Routing:
- net /ROW4: track 0.00 -> 266.1 mm
- net /ROW0: track 0.00 -> 260.3 mm
- net /ROW3: track 0.00 -> 242.3 mm
- net /ROW1: track 0.00 -> 233.4 mm
- net /ROW2: track 0.00 -> 204.5 mm
- net Net-(D61-A): track 0.00 -> 4.05 mm
- net Net-(D60-A): track 0.00 -> 4.05 mm
- net Net-(D13-A): track 0.00 -> 4.05 mm
- net Net-(D40-A): track 0.00 -> 4.05 mm
- net Net-(D51-A): track 0.00 -> 4.05 mm
- net Net-(D50-A): track 0.00 -> 4.05 mm
- net Net-(D48-A): track 0.00 -> 4.05 mm
- net Net-(D46-A): track 0.00 -> 4.05 mm
- net Net-(D54-A): track 0.00 -> 4.05 mm
- net Net-(D45-A): track 0.00 -> 4.05 mm
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
Commit message: Fix I2C bus
Parts:
- added C12: 4u7, Capacitor_SMD:C_0603_1608Metric, B.Cu at (132.2, 106.0)
- added C13: 100n, Capacitor_SMD:C_0603_1608Metric, B.Cu at (128.6, 106.0)
- added C14: 100n, Capacitor_SMD:C_0603_1608Metric, B.Cu at (125.0, 106.0)
- added U4: MCP23017_SO, Package_SO:SOIC-28W_7.5x17.9mm_P1.27mm, B.Cu at (101.0, 106.8)
- added U5: MCP23008-xSO, Package_SO:SOIC-18W_7.5x11.6mm_P1.27mm, B.Cu at (142.5, 115.2)
Connections:
- net /REC_USB_D+ renamed Net-(J1-D+-PadA6)
- net /REC_USB_D- renamed Net-(J1-D--PadA7)
- net Net-(U1-NRST) renamed /NRST
- U1 pad 10: /ROW0 -> /ROW_INT
- U1 pad 11: /ROW1 -> unconnected-(U1-PA1-Pad11)
- U1 pad 12: /ROW2 -> unconnected-(U1-PA2-Pad12)
- U1 pad 13: /ROW3 -> unconnected-(U1-PA3-Pad13)
- U1 pad 14: /ROW4 -> unconnected-(U1-PA4-Pad14)
- U1 pad 18: /Matrix/COL0 -> unconnected-(U1-PB0-Pad18)
- U1 pad 19: /Matrix/COL1 -> unconnected-(U1-PB1-Pad19)
- U1 pad 20: /Matrix/COL2 -> unconnected-(U1-PB2-Pad20)
- U1 pad 21: /Matrix/COL10 -> unconnected-(U1-PB10-Pad21)
- U1 pad 22: /Matrix/COL11 -> unconnected-(U1-PB11-Pad22)
- U1 pad 25: /Matrix/COL12 -> unconnected-(U1-PB12-Pad25)
- U1 pad 26: /Matrix/COL13 -> unconnected-(U1-PB13-Pad26)
- U1 pad 39: /Matrix/COL3 -> unconnected-(U1-PB3-Pad39)
- U1 pad 40: /Matrix/COL4 -> unconnected-(U1-PB4-Pad40)
- U1 pad 41: /Matrix/COL5 -> unconnected-(U1-PB5-Pad41)
- U1 pad 42: /Matrix/COL6 -> unconnected-(U1-PB6-Pad42)
- U1 pad 43: /Matrix/COL7 -> unconnected-(U1-PB7-Pad43)
- U1 pad 45: /Matrix/COL8 -> /I2C1_SCL
- U1 pad 46: /Matrix/COL9 -> /I2C1_SDA
Routing:
- net Net-(D34-A): track 0.00 -> 4.05 mm
Other:
- board outline added: 288.1 x 97.6 mm

Commit message: Reverse diodes on keyboard matrix
Parts:
- added R4: 2k2, Resistor_SMD:R_0603_1608Metric, F.Cu at (124.7, 112.2)
- added R5: 2k2, Resistor_SMD:R_0603_1608Metric, F.Cu at (124.7, 114.7)
- added R6: 10k, Resistor_SMD:R_0603_1608Metric, F.Cu at (124.7, 117.2)
- added R7: 10k, Resistor_SMD:R_0603_1608Metric, F.Cu at (124.7, 119.8)
- turned D1 to 90 degrees
- turned D10 to 90 degrees
- turned D11 to 90 degrees
- turned D12 to 90 degrees
- turned D13 to 90 degrees
- turned D14 to 90 degrees
- turned D15 to 90 degrees
- turned D16 to 90 degrees
- turned D17 to 90 degrees
- turned D18 to 90 degrees
- turned D19 to 90 degrees
- turned D2 to 90 degrees
- turned D20 to 90 degrees
- turned D21 to 90 degrees
- turned D22 to 90 degrees
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Connections:
- D1 pad 1: /ROW0 -> Net-(D1-K)
- D1 pad 2: Net-(D1-A) -> /ROW0
- D10 pad 1: /ROW0 -> Net-(D10-K)
- D10 pad 2: Net-(D10-A) -> /ROW0
- D11 pad 1: /ROW0 -> Net-(D11-K)
- D11 pad 2: Net-(D11-A) -> /ROW0
- D12 pad 1: /ROW0 -> Net-(D12-K)
- D12 pad 2: Net-(D12-A) -> /ROW0
- D13 pad 1: /ROW0 -> Net-(D13-K)
- D13 pad 2: Net-(D13-A) -> /ROW0
- D14 pad 1: /ROW0 -> Net-(D14-K)
- D14 pad 2: Net-(D14-A) -> /ROW0
- D15 pad 1: /ROW1 -> Net-(D15-K)
- D15 pad 2: Net-(D15-A) -> /ROW1
- D16 pad 1: /ROW1 -> Net-(D16-K)
- D16 pad 2: Net-(D16-A) -> /ROW1
- D17 pad 1: /ROW1 -> Net-(D17-K)
- D17 pad 2: Net-(D17-A) -> /ROW1
- D18 pad 1: /ROW1 -> Net-(D18-K)
- D18 pad 2: Net-(D18-A) -> /ROW1
- D19 pad 1: /ROW1 -> Net-(D19-K)
- D19 pad 2: Net-(D19-A) -> /ROW1
- D2 pad 1: /ROW0 -> Net-(D2-K)
- D2 pad 2: Net-(D2-A) -> /ROW0
- D20 pad 1: /ROW1 -> Net-(D20-K)
- D20 pad 2: Net-(D20-A) -> /ROW1
- D21 pad 1: /ROW1 -> Net-(D21-K)
- D21 pad 2: Net-(D21-A) -> /ROW1
- D22 pad 1: /ROW1 -> Net-(D22-K)
- D22 pad 2: Net-(D22-A) -> /ROW1
- D23 pad 1: /ROW1 -> Net-(D23-K)
- D23 pad 2: Net-(D23-A) -> /ROW1
- D24 pad 1: /ROW1 -> Net-(D24-K)
- D24 pad 2: Net-(D24-A) -> /ROW1
- D25 pad 1: /ROW1 -> Net-(D25-K)
- D25 pad 2: Net-(D25-A) -> /ROW1
- D26 pad 1: /ROW1 -> Net-(D26-K)
- D26 pad 2: Net-(D26-A) -> /ROW1
- D27 pad 1: /ROW1 -> Net-(D27-K)
- D27 pad 2: Net-(D27-A) -> /ROW1
- D28 pad 1: /ROW1 -> Net-(D28-K)
- D28 pad 2: Net-(D28-A) -> /ROW1
- D29 pad 1: /ROW2 -> Net-(D29-K)
- D29 pad 2: Net-(D29-A) -> /ROW2
- D3 pad 1: /ROW0 -> Net-(D3-K)
- D3 pad 2: Net-(D3-A) -> /ROW0
- D30 pad 1: /ROW2 -> Net-(D30-K)
- D30 pad 2: Net-(D30-A) -> /ROW2
- D31 pad 1: /ROW2 -> Net-(D31-K)
- D31 pad 2: Net-(D31-A) -> /ROW2
- D32 pad 1: /ROW2 -> Net-(D32-K)
- D32 pad 2: Net-(D32-A) -> /ROW2
- D33 pad 1: /ROW2 -> Net-(D33-K)
- D33 pad 2: Net-(D33-A) -> /ROW2
- D34 pad 1: /ROW2 -> Net-(D34-K)
- D34 pad 2: Net-(D34-A) -> /ROW2
- D35 pad 1: /ROW2 -> Net-(D35-K)
- D35 pad 2: Net-(D35-A) -> /ROW2
- D36 pad 1: /ROW2 -> Net-(D36-K)
- D36 pad 2: Net-(D36-A) -> /ROW2
- D37 pad 1: /ROW2 -> Net-(D37-K)
- D37 pad 2: Net-(D37-A) -> /ROW2
- D38 pad 1: /ROW2 -> Net-(D38-K)
- D38 pad 2: Net-(D38-A) -> /ROW2
- D39 pad 1: /ROW2 -> Net-(D39-K)
- D39 pad 2: Net-(D39-A) -> /ROW2
- D4 pad 1: /ROW0 -> Net-(D4-K)
- D4 pad 2: Net-(D4-A) -> /ROW0
- D40 pad 1: /ROW2 -> Net-(D40-K)
- D40 pad 2: Net-(D40-A) -> /ROW2
- D41 pad 1: /ROW2 -> Net-(D41-K)
- D41 pad 2: Net-(D41-A) -> /ROW2
- D42 pad 1: /ROW3 -> Net-(D42-K)
- D42 pad 2: Net-(D42-A) -> /ROW3
- D43 pad 1: /ROW3 -> Net-(D43-K)
- D43 pad 2: Net-(D43-A) -> /ROW3
- D44 pad 1: /ROW3 -> Net-(D44-K)
- D44 pad 2: Net-(D44-A) -> /ROW3
- D45 pad 1: /ROW3 -> Net-(D45-K)
- D45 pad 2: Net-(D45-A) -> /ROW3
- D46 pad 1: /ROW3 -> Net-(D46-K)
- D46 pad 2: Net-(D46-A) -> /ROW3
- D47 pad 1: /ROW3 -> Net-(D47-K)
- D47 pad 2: Net-(D47-A) -> /ROW3
- D48 pad 1: /ROW3 -> Net-(D48-K)
- D48 pad 2: Net-(D48-A) -> /ROW3
- D49 pad 1: /ROW3 -> Net-(D49-K)
- D49 pad 2: Net-(D49-A) -> /ROW3
- D5 pad 1: /ROW0 -> Net-(D5-K)
- D5 pad 2: Net-(D5-A) -> /ROW0
- D50 pad 1: /ROW3 -> Net-(D50-K)
- D50 pad 2: Net-(D50-A) -> /ROW3
- D51 pad 1: /ROW3 -> Net-(D51-K)
- D51 pad 2: Net-(D51-A) -> /ROW3
- D52 pad 1: /ROW3 -> Net-(D52-K)
- D52 pad 2: Net-(D52-A) -> /ROW3
- D53 pad 1: /ROW3 -> Net-(D53-K)
- D53 pad 2: Net-(D53-A) -> /ROW3
- D54 pad 1: /ROW4 -> Net-(D54-K)
- D54 pad 2: Net-(D54-A) -> /ROW4
- D55 pad 1: /ROW4 -> Net-(D55-K)
- D55 pad 2: Net-(D55-A) -> /ROW4
- D56 pad 1: /ROW4 -> Net-(D56-K)
- D56 pad 2: Net-(D56-A) -> /ROW4
- D57 pad 1: /ROW4 -> Net-(D57-K)
- D57 pad 2: Net-(D57-A) -> /ROW4
- D58 pad 1: /ROW4 -> Net-(D58-K)
- D58 pad 2: Net-(D58-A) -> /ROW4
- D59 pad 1: /ROW4 -> Net-(D59-K)
- D59 pad 2: Net-(D59-A) -> /ROW4
- D6 pad 1: /ROW0 -> Net-(D6-K)
- D6 pad 2: Net-(D6-A) -> /ROW0
- D60 pad 1: /ROW4 -> Net-(D60-K)
- D60 pad 2: Net-(D60-A) -> /ROW4
- D61 pad 1: /ROW4 -> Net-(D61-K)
- D61 pad 2: Net-(D61-A) -> /ROW4
- D7 pad 1: /ROW0 -> Net-(D7-K)
- D7 pad 2: Net-(D7-A) -> /ROW0
- D8 pad 1: /ROW0 -> Net-(D8-K)
- D8 pad 2: Net-(D8-A) -> /ROW0
- D9 pad 1: /ROW0 -> Net-(D9-K)
- D9 pad 2: Net-(D9-A) -> /ROW0
- SW1 pad 2: Net-(D1-A) -> Net-(D1-K)
- SW10 pad 2: Net-(D10-A) -> Net-(D10-K)
- SW11 pad 2: Net-(D11-A) -> Net-(D11-K)
- SW12 pad 2: Net-(D12-A) -> Net-(D12-K)
- SW13 pad 2: Net-(D13-A) -> Net-(D13-K)
- SW14 pad 2: Net-(D14-A) -> Net-(D14-K)
- SW15 pad 2: Net-(D15-A) -> Net-(D15-K)
- SW16 pad 2: Net-(D16-A) -> Net-(D16-K)
- SW17 pad 2: Net-(D17-A) -> Net-(D17-K)
- SW18 pad 2: Net-(D18-A) -> Net-(D18-K)
- SW19 pad 2: Net-(D19-A) -> Net-(D19-K)
- SW2 pad 2: Net-(D2-A) -> Net-(D2-K)
- SW20 pad 2: Net-(D20-A) -> Net-(D20-K)
- SW21 pad 2: Net-(D21-A) -> Net-(D21-K)
- SW22 pad 2: Net-(D22-A) -> Net-(D22-K)
- SW23 pad 2: Net-(D23-A) -> Net-(D23-K)
- SW24 pad 2: Net-(D24-A) -> Net-(D24-K)
- SW25 pad 2: Net-(D25-A) -> Net-(D25-K)
- SW26 pad 2: Net-(D26-A) -> Net-(D26-K)
- SW27 pad 2: Net-(D27-A) -> Net-(D27-K)
- SW28 pad 2: Net-(D28-A) -> Net-(D28-K)
- SW29 pad 2: Net-(D29-A) -> Net-(D29-K)
- SW3 pad 2: Net-(D3-A) -> Net-(D3-K)
- SW30 pad 2: Net-(D30-A) -> Net-(D30-K)
- SW31 pad 2: Net-(D31-A) -> Net-(D31-K)
- SW32 pad 2: Net-(D32-A) -> Net-(D32-K)
- SW33 pad 2: Net-(D33-A) -> Net-(D33-K)
- SW34 pad 2: Net-(D34-A) -> Net-(D34-K)
- SW35 pad 2: Net-(D35-A) -> Net-(D35-K)
- SW36 pad 2: Net-(D36-A) -> Net-(D36-K)
- SW37 pad 2: Net-(D37-A) -> Net-(D37-K)
- SW38 pad 2: Net-(D38-A) -> Net-(D38-K)
- SW39 pad 2: Net-(D39-A) -> Net-(D39-K)
- SW4 pad 2: Net-(D4-A) -> Net-(D4-K)
- SW40 pad 2: Net-(D40-A) -> Net-(D40-K)
- SW41 pad 2: Net-(D41-A) -> Net-(D41-K)
- SW42 pad 2: Net-(D42-A) -> Net-(D42-K)
- SW43 pad 2: Net-(D43-A) -> Net-(D43-K)
- SW44 pad 2: Net-(D44-A) -> Net-(D44-K)
- SW45 pad 2: Net-(D45-A) -> Net-(D45-K)
- SW46 pad 2: Net-(D46-A) -> Net-(D46-K)
- SW47 pad 2: Net-(D47-A) -> Net-(D47-K)
- SW48 pad 2: Net-(D48-A) -> Net-(D48-K)
- SW49 pad 2: Net-(D49-A) -> Net-(D49-K)
- SW5 pad 2: Net-(D5-A) -> Net-(D5-K)
- SW50 pad 2: Net-(D50-A) -> Net-(D50-K)
- SW51 pad 2: Net-(D51-A) -> Net-(D51-K)
- SW52 pad 2: Net-(D52-A) -> Net-(D52-K)
- SW53 pad 2: Net-(D53-A) -> Net-(D53-K)
- SW54 pad 2: Net-(D54-A) -> Net-(D54-K)
- SW55 pad 2: Net-(D55-A) -> Net-(D55-K)
- SW56 pad 2: Net-(D56-A) -> Net-(D56-K)
- SW57 pad 2: Net-(D57-A) -> Net-(D57-K)
- SW58 pad 2: Net-(D58-A) -> Net-(D58-K)
- SW59 pad 2: Net-(D59-A) -> Net-(D59-K)
- SW6 pad 2: Net-(D6-A) -> Net-(D6-K)
- SW60 pad 2: Net-(D60-A) -> Net-(D60-K)
- SW61 pad 2: Net-(D61-A) -> Net-(D61-K)
- SW7 pad 2: Net-(D7-A) -> Net-(D7-K)
- SW8 pad 2: Net-(D8-A) -> Net-(D8-K)
- SW9 pad 2: Net-(D9-A) -> Net-(D9-K)
Routing:
- net /ROW4: track 266.1 -> 0.00 mm
- net /Matrix/COL9: track 67.0 -> 333.1 mm
- net Net-(D61-K): track 0.00 -> 4.05 mm
- net Net-(D61-A): track 4.05 -> 0.00 mm
- net Net-(D60-K): track 0.00 -> 4.05 mm
- net Net-(D60-A): track 4.05 -> 0.00 mm
- net Net-(D13-K): track 0.00 -> 4.05 mm
- net Net-(D13-A): track 4.05 -> 0.00 mm
- net Net-(D40-K): track 0.00 -> 4.05 mm
- net Net-(D40-A): track 4.05 -> 0.00 mm
- net Net-(D51-K): track 0.00 -> 4.05 mm
- net Net-(D51-A): track 4.05 -> 0.00 mm
- net Net-(D50-K): track 0.00 -> 4.05 mm
- net Net-(D50-A): track 4.05 -> 0.00 mm
- net Net-(D48-K): track 0.00 -> 4.05 mm
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
Commit message: Clear board and add mounting holes
Parts:
- removed TP1, TP2: TestPoint, TestPoint:TestPoint_Pad_1.0x1.0mm
- added D63: LED, LED_SMD:LED_0201_0603Metric, F.Cu at (130.6, 154.8)
- added H1: MountingHole_Pad, Keyboard_Mounts:2.5mm, F.Cu at (52.6, 55.3)
- added H2: MountingHole_Pad, Keyboard_Mounts:2.5mm_Oblong, F.Cu at (166.7, 158.4)
- added H3: MountingHole_Pad, Keyboard_Mounts:2.5mm_Oblong, F.Cu at (166.7, 146.4)
- added H4: MountingHole_Pad, Keyboard_Mounts:2.5mm_Oblong, F.Cu at (176.2, 158.4)
- added H5: MountingHole_Pad, Keyboard_Mounts:2.5mm_Wide, F.Cu at (186.9, 147.6)
- added H6: MountingHole_Pad, Keyboard_Mounts:2.5mm_Wide, F.Cu at (189.3, 158.4)
- added J2: Conn_ARM_JTAG_SWD_10, Connector_PinHeader_1.27mm:PinHeader_2x05_P1.27mm_Horizontal, F.Cu at (113.2, 158.5)
- added R10: 10k, Resistor_SMD:R_0603_1608Metric, F.Cu at (123.0, 163.1)
- added R11: 330, Resistor_SMD:R_0603_1608Metric, F.Cu at (131.2, 152.7)
- added R8: 10k, Resistor_SMD:R_0603_1608Metric, F.Cu at (123.0, 158.1)
- added R9: 10k, Resistor_SMD:R_0603_1608Metric, F.Cu at (123.0, 160.6)
- C2: value 10u -> 4u7
- C8: value 10n -> 100n
Connections:
- U1 pad 16: unconnected-(U1-PA6-Pad16) -> Net-(U1-PA6)
- U1 pad 34: Net-(U1-PA13) -> /SWIO
- U1 pad 37: Net-(U1-PA14) -> /SWCLK
- U2 pad 5: +5V -> +3.3V
- U4 pad 15: +3.3V -> Net-(U4-A0)
- U4 pad 19: unconnected-(U4-INTB-Pad19) -> Net-(U4-INTB)
- U4 pad 20: unconnected-(U4-INTA-Pad20) -> Net-(U4-INTA)
Routing:
- net Net-(U1-PA14): track 7.55 -> 0.00 mm, vias 2 -> 0
- net /SWCLK: track 0.00 -> 7.55 mm, vias 0 -> 2
- net Net-(U1-PA13): track 6.00 -> 0.00 mm
- net /SWIO: track 0.00 -> 6.00 mm

Commit message: Routing almost complete
Parts:
- D63, J2, R10, R11, R4, R5, R6, R7, R8, R9: moved to B.Cu
- moved H5 170.3 mm to (28.6, 85.1)
- moved H3 151.5 mm to (288.6, 56.5)
- moved H6 144.3 mm to (313.6, 85.1)
- moved J2 123.0 mm to (36.1, 62.6), turned to 180 degrees
- moved R7 80.7 mm to (54.4, 80.2)
- moved H2 78.4 mm to (156.8, 80.6)
- moved R6 76.6 mm to (56.0, 83.3)
- moved R5 72.9 mm to (67.4, 69.6), turned to -90 degrees
- moved R4 72.7 mm to (65.8, 69.6), turned to -90 degrees
- moved R8 70.8 mm to (180.4, 116.6), turned to 180 degrees
- moved R10 70.8 mm to (180.4, 121.6), turned to 180 degrees
- moved R9 70.8 mm to (180.4, 119.1), turned to 180 degrees
- moved H4 61.8 mm to (219.1, 113.8)
- moved D63 59.1 mm to (172.8, 113.3), turned to 180 degrees
- moved R11 58.4 mm to (172.2, 111.1), turned to 180 degrees
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Connections:
- net Net-(J1-D--PadA7) renamed /USBC_D-
- J1 pad A6: Net-(J1-D+-PadA6) -> /USB_D+
- J1 pad B6: Net-(J1-D+-PadA6) -> /USB_D+
- U2 pad 3: Net-(J1-D+-PadA6) -> /USB_D+
Routing:
- net /Matrix/COL9: track 333.1 -> 67.0 mm
- net /ROW4: track 0.00 -> 209.9 mm, vias 0 -> 2
- net +3.3V: track 58.2 -> 174.8 mm, vias 0 -> 6
- net /I2C1_SCL: track 0.00 -> 69.0 mm, vias 0 -> 2
- net /I2C1_SDA: track 0.00 -> 68.7 mm
- net GND: track 0.00 -> 55.5 mm, vias 0 -> 52
- net /SWIO: track 6.00 -> 39.7 mm, vias 0 -> 2
- net /NRST: track 26.2 -> 59.1 mm, vias 2 -> 3
- net /SWCLK: track 7.55 -> 36.2 mm
- net /USB_D+: track 9.54 -> 37.2 mm
- net /ROW3: track 242.3 -> 266.0 mm, vias 0 -> 2
- net /ROW2: track 204.5 -> 223.5 mm
- net /ROW_INT: track 0.00 -> 16.0 mm, vias 0 -> 2
- net +5V: track 28.9 -> 14.5 mm
- net /USB_D-: track 10.4 -> 24.1 mm
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- added copper zone on B.Cu, net GND
- added copper zone on F.Cu, net GND

Commit message: Finished routing and various fixes
Parts:
- D63: moved to F.Cu
- moved D63 154.6 mm to (32.8, 47.6), turned to -90 degrees
- moved R11 134.1 mm to (46.8, 63.6)
- moved R8 51.3 mm to (130.4, 105.2), turned to 90 degrees
- moved R9 46.6 mm to (136.6, 103.2), turned to -90 degrees
- moved R10 46.0 mm to (138.2, 103.2), turned to -90 degrees
- moved C12 39.3 mm to (124.8, 103.2), turned to -90 degrees
- moved C13 32.2 mm to (123.2, 103.2), turned to -90 degrees
- moved C7 6.20 mm to (47.6, 79.4), turned to 180 degrees
- moved D57 6.05 mm to (156.0, 102.8)
- moved R1 4.24 mm to (57.6, 41.4)
- moved R2 4.24 mm to (57.6, 43.4)
- moved C14 3.05 mm to (138.6, 118.2), turned to 90 degrees
- moved C8 1.98 mm to (53.8, 76.4), turned to 180 degrees
- moved R4 1.22 mm to (64.6, 69.8)
- moved R5 1.22 mm to (66.2, 69.8)
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Connections:
- D15 pad 2: /ROW1 -> /ROW2
- J1 pad A6: /USB_D+ -> /USBC_D+
- J1 pad B6: /USB_D+ -> /USBC_D+
- U2 pad 3: /USB_D+ -> /USBC_D+
- U2 pad 5: +3.3V -> +5V
Routing:
- net /Matrix/COL13: track 89.0 -> 247.2 mm, vias 0 -> 2
- net /Matrix/COL12: track 81.1 -> 229.5 mm, vias 0 -> 3
- net /Matrix/COL11: track 85.5 -> 217.6 mm, vias 0 -> 3
- net /Matrix/COL10: track 96.3 -> 226.4 mm
- net /ROW2: track 223.5 -> 352.5 mm, vias 0 -> 10
- net /NRST: track 59.1 -> 185.6 mm, vias 3 -> 9
- net /Matrix/COL0: track 86.8 -> 207.9 mm
- net /Matrix/COL9: track 67.0 -> 169.9 mm
- net /Matrix/COL1: track 94.7 -> 191.5 mm, vias 4 -> 6
- net /ROW_INT: track 16.0 -> 110.1 mm, vias 2 -> 4
- net /ROW0: track 260.3 -> 350.3 mm, vias 0 -> 6
- net /Matrix/COL8: track 67.0 -> 152.2 mm
- net +3.3V: track 174.8 -> 249.7 mm, vias 6 -> 8
- net /Matrix/COL2: track 91.0 -> 158.8 mm, vias 0 -> 2
- net /ROW1: track 233.4 -> 300.8 mm, vias 0 -> 4
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
Commit message: Finished routing and various fixes
Routing:
- net GND: vias 86 -> 88
Changed lines of the file:
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@@
 	)
 	(via
+		(at 57.584375 29.384375)
+		(size 0.8)
+		(drill 0.3)
+		(layers "F.Cu" "B.Cu")
+		(net 2)
+	)
+	(via
 		(at 81.184375 100.984375)
 		(size 0.8)
@@
 	)
 	(via
+		(at 39.784375 29.384375)
+		(size 0.8)
+		(drill 0.3)
+		(layers "F.Cu" "B.Cu")
+		(net 2)
+	)
+	(via
 		(at 32.784375 46.184375)
 		(size 0.8)
@@
 	)
 	(segment
-		(start 146.784375 121.384375)
-		(end 134.584375 121.384375)
-		(width 0.2)
-		(layer "F.Cu")
-		(net 81)
-	)
-	(segment
-		(start 116.184375 94.384375)
-		(end 115.2525 93.4525)
+		(start 116.184375 98.184375)
+		(end 116.184375 94.384375)
 		(width 0.2)
 		(layer "F.Cu")
@@
 	)
 	(segment
-		(start 128.584375 115.384375)
-		(end 128.584375 110.184375)
+		(start 116.184375 94.384375)
+		(end 115.2525 93.4525)
 		(width 0.2)
 		(layer "F.Cu")
@@
 	)
 	(segment
-		(start 134.584375 121.384375)
-		(end 128.584375 115.384375)
+		(start 146.784375 121.384375)
+		(end 134.584375 121.384375)
 		(width 0.2)
 		(layer "F.Cu")
@@
 	)
 	(segment
-		(start 105.7275 73.66)
-		(end 105.7275 83.185)
+		(start 128.584375 115.384375)
+		(end 128.584375 110.584375)
 		(width 0.2)
 		(layer "F.Cu")
@@
 	)
 	(segment
-		(start 116.184375 97.784375)
-		(end 116.184375 94.384375)
+		(start 105.7275 73.66)
+		(end 105.7275 83.185)
 		(width 0.2)
 		(layer "F.Cu")
@@
 	)
 	(segment
+		(start 128.584375 110.584375)
+		(end 116.184375 98.184375)
+		(width 0.2)
+		(layer "F.Cu")
+		(net 81)
+	)
+	(segment
 		(start 100.965 68.8975)
 		(end 105.7275 73.66)
@@
 	)
 	(segment
-		(start 128.584375 110.184375)
-		(end 116.184375 97.784375)
+		(start 134.584375 121.384375)
+		(end 128.584375 115.384375)
 		(width 0.2)
 		(layer "F.Cu")
