File: pcb/simplekeyboard.kicad_sch (KiCad schematic)
At the start: 42 parts, among them J1 USB_C_Receptacle_USB2.0_16P, J2 Conn_ARM_JTAG_SWD_10, SW62 SW_SPDT, SW63 SW_Push, U1 STM32F072CBT6, U2 USBLC6-2SC6, U3 LD39050PU33R, U4 MCP23017_SO, U5 MCP23008-xSO

Commit message: Cleanup silkscreen
Other:
- moved on the sheet: C14, U5

Commit message: Fixed critical mistake where CAPSLOCK and Tab were indistinguishable
Connections:
- net SWIO renamed SWDIO
Changed lines of the file:
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@@
 		)
 	)
-	(label "SWIO"
+	(label "SWDIO"
 		(at 193.04 123.19 0)
 		(effects
@@
 		)
 	)
-	(label "SWIO"
+	(label "SWDIO"
 		(at 83.82 140.97 0)
 		(effects

Commit message: Changed a few footrpints
Parts:
- C10, C11, C13, C14, C3, C4, C5, C8: footprint Capacitor_SMD:C_0603_1608Metric -> Capacitor_SMD:C_0402_1005Metric
- D63: footprint LED_SMD:LED_0201_0603Metric -> LED_SMD:LED_0603_1608Metric
- H5, H6: footprint Keyboard_Mounts:2.5mm_Wide -> Keyboard_Mounts:2.5mm_Oblong
- R1, R2, R3: footprint Resistor_SMD:R_0805_2012Metric -> Resistor_SMD:R_0603_1608Metric
Changed lines of the file:
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@@
 			)
 		)
-		(property "Footprint" "Resistor_SMD:R_0805_2012Metric"
+		(property "Footprint" "Resistor_SMD:R_0603_1608Metric"
 			(at 54.102 41.91 90)
 			(effects
@@
 			)
 		)
-		(property "Footprint" "Capacitor_SMD:C_0603_1608Metric"
+		(property "Footprint" "Capacitor_SMD:C_0402_1005Metric"
 			(at 38.1 94.2848 0)
 			(effects
@@
 			)
 		)
-		(property "Footprint" "LED_SMD:LED_0201_0603Metric"
+		(property "Footprint" "LED_SMD:LED_0603_1608Metric"
 			(at 99.06 123.19 0)
 			(effects
@@
 			)
 		)
-		(property "Footprint" "Capacitor_SMD:C_0603_1608Metric"
+		(property "Footprint" "Capacitor_SMD:C_0402_1005Metric"
 			(at 129.2352 146.05 0)
 			(effects
@@
 			)
 		)
-		(property "Footprint" "Capacitor_SMD:C_0603_1608Metric"
+		(property "Footprint" "Capacitor_SMD:C_0402_1005Metric"
 			(at 162.2552 31.75 0)
 			(effects
@@
 			)
 		)
-		(property "Footprint" "Capacitor_SMD:C_0603_1608Metric"
+		(property "Footprint" "Capacitor_SMD:C_0402_1005Metric"
 			(at 237.1852 34.29 0)
 			(effects
@@
 			)
 		)
-		(property "Footprint" "Capacitor_SMD:C_0603_1608Metric"
+		(property "Footprint" "Capacitor_SMD:C_0402_1005Metric"
 			(at 149.5552 123.19 0)
 			(effects
@@
 			)
 		)
-		(property "Footprint" "Capacitor_SMD:C_0603_1608Metric"
+		(property "Footprint" "Capacitor_SMD:C_0402_1005Metric"
 			(at 139.3952 146.05 0)
 			(effects
@@
 			)
 		)
-		(property "Footprint" "Resistor_SMD:R_0805_2012Metric"
+		(property "Footprint" "Resistor_SMD:R_0603_1608Metric"
 			(at 41.91 114.808 90)
 			(effects
@@
 			)
 		)
-		(property "Footprint" "Keyboard_Mounts:2.5mm_Wide"
+		(property "Footprint" "Keyboard_Mounts:2.5mm_Oblong"
 			(at 127 215.9 0)
 			(effects
@@
 			)
 		)
-		(property "Footprint" "Capacitor_SMD:C_0603_1608Metric"
+		(property "Footprint" "Capacitor_SMD:C_0402_1005Metric"
 			(at 129.2352 123.19 0)
 			(effects
@@
 			)
 		)
-		(property "Footprint" "Resistor_SMD:R_0805_2012Metric"
+		(property "Footprint" "Resistor_SMD:R_0603_1608Metric"
 			(at 60.452 41.91 90)
 			(effects
@@
 			)
 		)
-		(property "Footprint" "Keyboard_Mounts:2.5mm_Wide"
+		(property "Footprint" "Keyboard_Mounts:2.5mm_Oblong"
 			(at 104.14 215.9 0)
 			(effects
@@
 			)
 		)
-		(property "Footprint" "Capacitor_SMD:C_0603_1608Metric"
+		(property "Footprint" "Capacitor_SMD:C_0402_1005Metric"
 			(at 119.0752 146.05 0)
 			(effects

Commit message: Changed schematic header
Other:
- company: (none) -> agrantushinsky/simplekeyboard
- title: simplekeyboard -> Main
Changed lines of the file:
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@@
 	(paper "A4")
 	(title_block
-		(title "simplekeyboard")
-		(date "2026-05-05")
+		(title "Main")
+		(date "2026-07-18")
 		(rev "A")
+		(company "agrantushinsky/simplekeyboard")
 	)
 	(rectangle

Commit message: Fixed diode orientation and SDA/SCL
Connections:
- net I2C1_SCL: now also U4.12 (SCK); no longer U4.13 (SDA)
- net I2C1_SDA: now also U4.13 (SDA); no longer U4.12 (SCK)
Changed lines of the file:
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@@
 		(title "Main")
 		(date "2026-07-18")
-		(rev "A")
+		(rev "1.1")
 		(company "agrantushinsky/simplekeyboard")
 	)
@@
 		)
 	)
+	(label "I2C1_SCL"
+		(at 132.08 44.45 180)
+		(effects
+			(font
+				(size 1.27 1.27)
+			)
+			(justify right bottom)
+		)
+	)
 	(label "USBC_D-"
 		(at 53.34 60.96 0)
@@
 		)
 	)
+	(label "I2C1_SDA"
+		(at 132.08 41.91 180)
+		(effects
+			(font
+				(size 1.27 1.27)
+			)
+			(justify right bottom)
+		)
+	)
 	(label "VDDIO2"
 		(at 139.7 114.3 0)
@@
 		)
 	)
-	(label "I2C1_SCL"
-		(at 132.08 41.91 180)
-		(effects
-			(font
-				(size 1.27 1.27)
-			)
-			(justify right bottom)
-		)
-	)
 	(label "SWCLK"
 		(at 83.82 143.51 0)
@@
 		)
 	)
-	(label "I2C1_SDA"
-		(at 132.08 44.45 180)
-		(effects
-			(font
-				(size 1.27 1.27)
-			)
-			(justify right bottom)
-		)
-	)
